File: pi.kicad_sch (KiCad schematic)
At the start: 30 parts, among them J2 RPi GPIO 2x20, J6 PI_CONSOLE, Q1 HYG032N03LR1C1, U18 SP3232EEN-L/TR, U19 LM74700QDBVRQ1, U21 24LC32A-I/SN

Commit message: Add LCSC order lists; give J6/J7 headers an LCSC number
- tools/lcsc_order.py: LCSC BOM Tool upload lists for N boards (all parts, and
  through-hole-only for when JLCPCB assembles the SMD side)
- J6/J7 1x3 2.54 mm headers: C49257

Co-Authored-By: Claude Opus 5.5 (1M context) <noreply@anthropic.com>
Parts:
- J6: LCSC (none) -> C49257
Changed lines of the file:
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@@
+			)
+		)
+		(property "LCSC" "C49257"
+			(at 369.57 240.03 0)
+			(hide yes)
+			(show_name no)
+			(do_not_autoplace no)
+			(effects
+				(font
+					(size 1.27 1.27)
+				)
 			)
 		)

Commit message: Replace parts LCSC has on backorder with in-stock equivalents
47k C111134, 1k C22548, 240R C114613, 243k C403098, 1uF C91185, 22uF C77091,
LM74700QDBVTQ1 C2653623, TMPC1265HP-100MG-D C305223 (L1), AON7524 C431195 (Q1).
Same values, packages and land patterns. The JLCPCB assembly BOM keeps the four
JLC Basic originals that JLCPCB itself still stocks.

Co-Authored-By: Claude Opus 5.5 (1M context) <noreply@anthropic.com>
Parts:
- Q1: value HYG032N03LR1C1 -> AON7524; LCSC C2827233 -> C431195
- U19: value LM74700QDBVRQ1 -> LM74700QDBVTQ1; LCSC C2941042 -> C2653623
Other:
- note added: "IDEAL DIODE: LM74700-Q1 + AON7524 (30 V, 3.3 mOhm) blocks back-feed from the Pi's own USB-C. C24 (VCAP) connects to ANODE per the LM74700 datasheet; rated >= 25 V. 100 nF = 2.3 ms turn-on delay. BRING-UP: 3.3 mOhm is below TI's 8-20 mOhm window - scope the gate with the Pi idling for hunting."
- note removed: "IDEAL DIODE: LM74700-Q1 + HYG032N03LR1C1 (30 V, 3.3 mOhm) blocks back-feed from the Pi's own USB-C. C24 (VCAP) connects to ANODE per the LM74700 datasheet; rated >= 25 V. 100 nF = 2.3 ms turn-on delay. BRING-UP: 3.3 mOhm is below TI's 8-20 mOhm window - scope the gate with the Pi idling for hunting."
Changed lines of the file:
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@@
 		)
 	)
-	(text "IDEAL DIODE: LM74700-Q1 + HYG032N03LR1C1 (30 V, 3.3 mOhm) blocks back-feed from the Pi's own USB-C.\nC24 (VCAP) connects to ANODE per the LM74700 datasheet; rated >= 25 V. 100 nF = 2.3 ms turn-on delay.\nBRING-UP: 3.3 mOhm is below TI's 8-20 mOhm window - scope the gate with the Pi idling for hunting."
+	(text "IDEAL DIODE: LM74700-Q1 + AON7524 (30 V, 3.3 mOhm) blocks back-feed from the Pi's own USB-C.\nC24 (VCAP) connects to ANODE per the LM74700 datasheet; rated >= 25 V. 100 nF = 2.3 ms turn-on delay.\nBRING-UP: 3.3 mOhm is below TI's 8-20 mOhm window - scope the gate with the Pi idling for hunting."
 		(exclude_from_sim no)
 		(at 170 22 0)
@@
 			)
 		)
-		(property "Value" "HYG032N03LR1C1"
+		(property "Value" "AON7524"
 			(at 229.87 67.31 90)
 			(show_name no)
@@
 			)
 		)
-		(property "LCSC" "C2827233"
+		(property "LCSC" "C431195"
 			(at 229.87 59.69 90)
 			(hide yes)
@@
 			)
 		)
-		(property "Value" "LM74700QDBVRQ1"
+		(property "Value" "LM74700QDBVTQ1"
 			(at 237.49 99.06 0)
 			(show_name no)
@@
 			)
 		)
-		(property "LCSC" "C2941042"
+		(property "LCSC" "C2653623"
 			(at 229.87 90.17 0)
 			(hide yes)
