File: power.kicad_sch (KiCad schematic)
At the start: 53 parts, among them J3 PWR_CHAIN, J4 PWR_CHAIN, Q2 IRFR5305TRPBF, U7 LM317, U8 TPS54560BDDAR, U9 TPS54360BDDAR

Commit message: Replace parts LCSC has on backorder with in-stock equivalents
47k C111134, 1k C22548, 240R C114613, 243k C403098, 1uF C91185, 22uF C77091,
LM74700QDBVTQ1 C2653623, TMPC1265HP-100MG-D C305223 (L1), AON7524 C431195 (Q1).
Same values, packages and land patterns. The JLCPCB assembly BOM keeps the four
JLC Basic originals that JLCPCB itself still stocks.

Co-Authored-By: Claude Opus 5.5 (1M context) <noreply@anthropic.com>
Parts:
- C10, C11, C17, C18, C19, C8, C9: LCSC C12891 -> C77091
- C20: LCSC C28323 -> C91185
- L1: LCSC C840531 -> C305223; MPN SRP1265A-100M -> TMPC1265HP-100MG-D
- R1, R5: LCSC C23351 -> C403098
- R9: LCSC C23350 -> C114613
Changed lines of the file:
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@@
 			)
 		)
-		(property "LCSC" "C12891"
+		(property "LCSC" "C77091"
 			(at 351.79 214.63 0)
 			(hide yes)
@@
 			)
 		)
-		(property "LCSC" "C12891"
+		(property "LCSC" "C77091"
 			(at 193.04 214.63 0)
 			(hide yes)
@@
 			)
 		)
-		(property "LCSC" "C12891"
+		(property "LCSC" "C77091"
 			(at 172.72 214.63 0)
 			(hide yes)
@@
 			)
 		)
-		(property "LCSC" "C12891"
+		(property "LCSC" "C77091"
 			(at 361.95 214.63 0)
 			(hide yes)
@@
 			)
 		)
-		(property "LCSC" "C12891"
+		(property "LCSC" "C77091"
 			(at 182.88 214.63 0)
 			(hide yes)
@@
 			)
 		)
-		(property "LCSC" "C840531"
+		(property "LCSC" "C305223"
 			(at 111.76 214.63 0)
 			(hide yes)
@@
 			)
 		)
-		(property "MPN" "SRP1265A-100M"
+		(property "MPN" "TMPC1265HP-100MG-D"
 			(at 111.76 214.63 0)
 			(hide yes)
@@
 			)
 		)
-		(property "LCSC" "C23351"
+		(property "LCSC" "C403098"
 			(at 240.03 214.63 0)
 			(hide yes)
@@
 			)
 		)
-		(property "LCSC" "C12891"
+		(property "LCSC" "C77091"
 			(at 372.11 214.63 0)
 			(hide yes)
@@
 			)
 		)
-		(property "LCSC" "C23351"
+		(property "LCSC" "C403098"
 			(at 50.8 214.63 0)
 			(hide yes)
@@
 			)
 		)
-		(property "LCSC" "C23350"
+		(property "LCSC" "C114613"
 			(at 309.88 100.33 0)
 			(hide yes)
@@
 			)
 		)
-		(property "LCSC" "C12891"
+		(property "LCSC" "C77091"
 			(at 162.56 214.63 0)
 			(hide yes)
@@
 			)
 		)
-		(property "LCSC" "C28323"
+		(property "LCSC" "C91185"
 			(at 299.72 100.33 0)
 			(hide yes)
