File: usb-console-server.kicad_pcb (KiCad board)
At the start: 4 copper layers, 138 x 141 mm, 320 parts, among them J1 USB-C, J2 RPi GPIO 2x20, J3 PWR_CHAIN, J4 PWR_CHAIN, J5 HC-RJ45-059D-2x8-2-04, J6 PI_CONSOLE, J7 UPDI, J8 LINK, J9 LINK, Q1 HYG032N03LR1C1, Q2 IRFR5305TRPBF, U1 FT4232HL, U10 MAX3232EIDR, U11 MAX3232EIDR, U12 MAX3232EIDR, U13 MAX3232EIDR, U14 MAX3232EIDR, U15 MAX3232EIDR, U16 MAX3232EIDR, U17 MAX3232EIDR, U18 SP3232EEN-L/TR, U19 LM74700QDBVRQ1, U2 FT4232HL, U20 24LC02B-I/SN, U21 24LC32A-I/SN, U22 PRTR5V0U2F, U3 FT4232HL, U31 93LC46BT-I/SN, U32 93LC46BT-I/SN, U33 93LC46BT-I/SN, U34 93LC46BT-I/SN, U4 FT4232HL, U5 USB2514BI-AEZG-TR, U6 ATtiny3216-SN, U7 LM317, U8 TPS54560BDDAR, U9 TPS54360BDDAR, X1 24MHz, X2 12MHz, X3 12MHz, X4 12MHz, X5 12MHz

Commit message: Replace parts LCSC has on backorder with in-stock equivalents
47k C111134, 1k C22548, 240R C114613, 243k C403098, 1uF C91185, 22uF C77091,
LM74700QDBVTQ1 C2653623, TMPC1265HP-100MG-D C305223 (L1), AON7524 C431195 (Q1).
Same values, packages and land patterns. The JLCPCB assembly BOM keeps the four
JLC Basic originals that JLCPCB itself still stocks.

Co-Authored-By: Claude Opus 5.5 (1M context) <noreply@anthropic.com>
Parts:
- Q1: value HYG032N03LR1C1 -> AON7524
- U19: value LM74700QDBVRQ1 -> LM74700QDBVTQ1
Changed lines of the file:
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@@
 			)
 		)
-		(property "Value" "LM74700QDBVRQ1"
+		(property "Value" "LM74700QDBVTQ1"
 			(at 0 2.4 0)
 			(layer "F.Fab")
@@
 			)
 		)
-		(property "LCSC" "C2941042"
+		(property "LCSC" "C2653623"
 			(at 0 0 0)
 			(layer "F.Fab")
@@
 			)
 		)
-		(property "LCSC" "C12891"
+		(property "LCSC" "C77091"
 			(at 0 0 0)
 			(layer "F.Fab")
@@
 			)
 		)
-		(property "LCSC" "C12891"
+		(property "LCSC" "C77091"
 			(at 0 0 90)
 			(layer "F.Fab")
@@
 			)
 		)
-		(property "LCSC" "C840531"
+		(property "LCSC" "C305223"
 			(at 0 0 0)
 			(layer "F.Fab")
@@
 			)
 		)
-		(property "MPN" "SRP1265A-100M"
+		(property "MPN" "TMPC1265HP-100MG-D"
 			(at 0 0 0)
 			(layer "F.Fab")
@@
 			)
 		)
-		(property "LCSC" "C23350"
+		(property "LCSC" "C114613"
 			(at 0 0 0)
 			(layer "F.Fab")
@@
 			)
 		)
-		(property "LCSC" "C12891"
+		(property "LCSC" "C77091"
 			(at 0 0 0)
 			(layer "F.Fab")
@@
 			)
 		)
-		(property "LCSC" "C25819"
+		(property "LCSC" "C111134"
 			(at 0 0 90)
 			(layer "F.Fab")
@@
 			)
 		)
-		(property "LCSC" "C12891"
+		(property "LCSC" "C77091"
 			(at 0 0 90)
 			(layer "F.Fab")
@@
 			)
 		)
-		(property "Value" "HYG032N03LR1C1"
+		(property "Value" "AON7524"
 			(at 0 5.4 0)
 			(layer "F.Fab")
@@
 			)
 		)
-		(property "LCSC" "C2827233"
+		(property "LCSC" "C431195"
 			(at 0 0 0)
 			(layer "F.Fab")
@@
 			)
 		)
-		(property "LCSC" "C23351"
+		(property "LCSC" "C403098"
 			(at 0 0 0)
 			(layer "F.Fab")
@@
 			)
 		)
-		(property "LCSC" "C28323"
+		(property "LCSC" "C91185"
 			(at 0 0 90)
 			(layer "F.Fab")
@@
 			)
 		)
-		(property "LCSC" "C25819"
+		(property "LCSC" "C111134"
 			(at 0 0 0)
 			(layer "F.Fab")
@@
 			)
 		)
-		(property "LCSC" "C23351"
+		(property "LCSC" "C403098"
 			(at 0 0 0)
 			(layer "F.Fab")
@@
 			)
 		)
-		(property "LCSC" "C28323"
+		(property "LCSC" "C91185"
 			(at 0 0 0)
 			(layer "F.Fab")
@@
 			)
 		)
-		(property "LCSC" "C12891"
+		(property "LCSC" "C77091"
 			(at 0 0 90)
 			(layer "F.Fab")
@@
 			)
 		)
-		(property "LCSC" "C12891"
+		(property "LCSC" "C77091"
 			(at 0 0 0)
 			(layer "F.Fab")
@@
 			)
 		)
-		(property "LCSC" "C21190"
+		(property "LCSC" "C22548"
 			(at 0 0 0)
 			(layer "F.Fab")
@@
 			)
 		)
-		(property "LCSC" "C12891"
+		(property "LCSC" "C77091"
 			(at 0 0 90)
 			(layer "F.Fab")
@@
 			)
 		)
-		(property "LCSC" "C12891"
+		(property "LCSC" "C77091"
 			(at 0 0 0)
 			(layer "F.Fab")
