File: hub.kicad_sch (KiCad schematic)
At the start: 42 parts, among them J1 USB-C, U20 24LC02B-I/SN, U22 PRTR5V0U2F, U5 USB2514BI-AEZG-TR, X1 24MHz

Commit message: Replace parts LCSC has on backorder with in-stock equivalents
47k C111134, 1k C22548, 240R C114613, 243k C403098, 1uF C91185, 22uF C77091,
LM74700QDBVTQ1 C2653623, TMPC1265HP-100MG-D C305223 (L1), AON7524 C431195 (Q1).
Same values, packages and land patterns. The JLCPCB assembly BOM keeps the four
JLC Basic originals that JLCPCB itself still stocks.

Co-Authored-By: Claude Opus 5.5 (1M context) <noreply@anthropic.com>
Parts:
- C174: LCSC C28323 -> C91185
- R18: LCSC C25819 -> C111134
Changed lines of the file:
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@@
 			)
 		)
-		(property "LCSC" "C28323"
+		(property "LCSC" "C91185"
 			(at 40.64 124.46 0)
 			(hide yes)
@@
 			)
 		)
-		(property "LCSC" "C25819"
+		(property "LCSC" "C111134"
 			(at 50.8 124.46 0)
 			(hide yes)

Commit message: Use in-stock 24 MHz crystal (C5444545) and green LED (C12065); add 5-board LCSC list
Both originals (C70590, C72043) are out of stock at LCSC; the replacements have the
same spec and package. Adds usb-console-server_lcsc_order_5boards.csv and a small
add-missing list for the cart.

Co-Authored-By: Claude Opus 5.5 (1M context) <noreply@anthropic.com>
Parts:
- X1: LCSC C70590 -> C5444545
Changed lines of the file:
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@@
 			)
 		)
-		(property "LCSC" "C70590"
+		(property "LCSC" "C5444545"
 			(at 299.72 100.33 0)
 			(hide yes)
