File: mcu.kicad_sch (KiCad schematic)
At the start: 30 parts, among them J7 UPDI, J8 LINK, J9 LINK, U6 ATtiny3216-SN

Commit message: Add LCSC order lists; give J6/J7 headers an LCSC number
- tools/lcsc_order.py: LCSC BOM Tool upload lists for N boards (all parts, and
  through-hole-only for when JLCPCB assembles the SMD side)
- J6/J7 1x3 2.54 mm headers: C49257

Co-Authored-By: Claude Opus 5.5 (1M context) <noreply@anthropic.com>
Parts:
- J7: LCSC (none) -> C49257
Changed lines of the file:
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@@
+			)
+		)
+		(property "LCSC" "C49257"
+			(at 39.37 74.93 0)
+			(hide yes)
+			(show_name no)
+			(do_not_autoplace no)
+			(effects
+				(font
+					(size 1.27 1.27)
+				)
 			)
 		)

Commit message: Replace parts LCSC has on backorder with in-stock equivalents
47k C111134, 1k C22548, 240R C114613, 243k C403098, 1uF C91185, 22uF C77091,
LM74700QDBVTQ1 C2653623, TMPC1265HP-100MG-D C305223 (L1), AON7524 C431195 (Q1).
Same values, packages and land patterns. The JLCPCB assembly BOM keeps the four
JLC Basic originals that JLCPCB itself still stocks.

Co-Authored-By: Claude Opus 5.5 (1M context) <noreply@anthropic.com>
Parts:
- C53: LCSC C12891 -> C77091
- R27: LCSC C25819 -> C111134
- R42: LCSC C21190 -> C22548
Changed lines of the file:
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@@
 			)
 		)
-		(property "LCSC" "C25819"
+		(property "LCSC" "C111134"
 			(at 175.26 54.61 0)
 			(hide yes)
@@
 			)
 		)
-		(property "LCSC" "C21190"
+		(property "LCSC" "C22548"
 			(at 271.78 139.7 0)
 			(hide yes)
@@
 			)
 		)
-		(property "LCSC" "C12891"
+		(property "LCSC" "C77091"
 			(at 205.74 54.61 0)
 			(hide yes)

Commit message: Use in-stock 24 MHz crystal (C5444545) and green LED (C12065); add 5-board LCSC list
Both originals (C70590, C72043) are out of stock at LCSC; the replacements have the
same spec and package. Adds usb-console-server_lcsc_order_5boards.csv and a small
add-missing list for the cart.

Co-Authored-By: Claude Opus 5.5 (1M context) <noreply@anthropic.com>
Parts:
- D6: LCSC C72043 -> C12065
Changed lines of the file:
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@@
 			)
 		)
-		(property "LCSC" "C72043"
+		(property "LCSC" "C12065"
 			(at 287.02 149.86 90)
 			(hide yes)
